Commit message: Add obj files

File: config_folder/robot_files/stretch_description_SE3_eoa_wrist_dw3_tool_sg3.urdf (robot description, URDF)
Before this commit: robot stretch, 52 links, 51 joints
Links:
- link base_imu: geometry collision mesh filename=./stretch_objs/base_imu.obj; visual mesh filename=./stretch_objs/base_imu.obj
- link base_link: geometry collision mesh filename=./stretch_objs/base_link_collision.obj; visual mesh filename=./stretch_objs/base_link.obj
- link camera_link: geometry collision box size=0.02505 0.09 0.025; visual mesh filename=./stretch_objs/d435.obj
- link caster_link: geometry collision sphere radius=0.032; visual mesh filename=./stretch_objs/omni_wheel_m.obj
- link laser: geometry collision mesh filename=./stretch_objs/laser_collision.obj; visual mesh filename=./stretch_objs/laser.obj
- link link_arm_l0: geometry collision mesh filename=./stretch_objs/link_arm_l0_collision.obj; visual mesh filename=./stretch_objs/link_arm_l0.obj
- link link_arm_l1: geometry collision mesh filename=./stretch_objs/link_arm_l1_collision.obj; visual mesh filename=./stretch_objs/link_arm_l1.obj
- link link_arm_l2: geometry collision mesh filename=./stretch_objs/link_arm_l2_collision.obj; visual mesh filename=./stretch_objs/link_arm_l2.obj
- link link_arm_l3: geometry collision mesh filename=./stretch_objs/link_arm_l3_collision.obj; visual mesh filename=./stretch_objs/link_arm_l3.obj
- link link_arm_l4: geometry collision mesh filename=./stretch_objs/link_arm_l4_collision.obj; visual mesh filename=./stretch_objs/link_arm_l4.obj
- link link_aruco_d405: geometry collision mesh filename=./stretch_objs/link_SG3_aruco_d405.obj; visual mesh filename=./stretch_objs/link_SG3_aruco_d405.obj
- link link_aruco_fingertip_left: geometry collision mesh filename=./stretch_objs/link_SG3_aruco_fingertip_left.obj; visual mesh filename=./stretch_objs/link_SG3_aruco_fingertip_left.obj
- link link_aruco_fingertip_right: geometry collision mesh filename=./stretch_objs/link_SG3_aruco_fingertip_right.obj; visual mesh filename=./stretch_objs/link_SG3_aruco_fingertip_right.obj
- link link_aruco_inner_wrist: geometry collision mesh filename=./stretch_objs/link_aruco_inner_wrist.obj; visual mesh filename=./stretch_objs/link_aruco_inner_wrist.obj
- link link_aruco_left_base: geometry collision mesh filename=./stretch_objs/link_aruco_left_base.obj; visual mesh filename=./stretch_objs/link_aruco_left_base.obj
- link link_aruco_right_base: geometry collision mesh filename=./stretch_objs/link_aruco_right_base.obj; visual mesh filename=./stretch_objs/link_aruco_right_base.obj
- link link_aruco_shoulder: geometry collision mesh filename=./stretch_objs/link_aruco_shoulder.obj; visual mesh filename=./stretch_objs/link_aruco_shoulder.obj
- link link_aruco_top_wrist: geometry collision mesh filename=./stretch_objs/link_aruco_top_wrist.obj; visual mesh filename=./stretch_objs/link_aruco_top_wrist.obj
- link link_gripper_finger_left: geometry collision mesh filename=./stretch_objs/link_SG3_gripper_finger_left_collision.obj; visual mesh filename=./stretch_objs/link_SG3_gripper_finger_left.obj
- link link_gripper_finger_right: geometry collision mesh filename=./stretch_objs/link_SG3_gripper_finger_right_collision.obj; visual mesh filename=./stretch_objs/link_SG3_gripper_finger_right.obj
- link link_gripper_fingertip_left: geometry collision mesh filename=./stretch_objs/link_SG3_gripper_fingertip_left_collision.obj; visual mesh filename=./stretch_objs/link_SG3_gripper_fingertip_left.obj
- link link_gripper_fingertip_right: geometry collision mesh filename=./stretch_objs/link_SG3_gripper_fingertip_right_collision.o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; visual mesh filename=./stretch_objs/link_SG3_gripper_fingertip_right.obj
- link link_gripper_s3_body: geometry collision mesh filename=./stretch_objs/link_SG3_gripper_body_collision.obj; visual mesh filename=./stretch_objs/link_SG3_gripper_body.obj
- link link_ground: geometry collision mesh filename=./stretch_objs/link_ground_collision.obj; visual mesh filename=./stretch_objs/link_ground_collision.obj
- link link_head: geometry collision mesh filename=./stretch_objs/link_head_collision.obj; visual mesh filename=./stretch_objs/link_head.obj
- link link_head_nav_cam: geometry collision mesh filename=./stretch_objs/link_SE3_head_nav_cam_collision.obj; visual mesh filename=./stretch_objs/link_SE3_head_nav_cam.obj
- link link_head_pan: geometry collision mesh filename=./stretch_objs/link_head_pan_collision.obj; visual mesh filename=./stretch_objs/link_head_pan.obj
- link link_head_tilt: geometry collision mesh filename=./stretch_objs/link_head_tilt_collision.obj; visual mesh filename=./stretch_objs/link_head_tilt.obj
- link link_left_wheel: geometry collision mesh filename=./stretch_objs/link_left_wheel_collision.obj; visual mesh filename=./stretch_objs/link_left_wheel.obj
- link link_lift: geometry collision mesh filename=./stretch_objs/link_lift_collision.obj; visual mesh filename=./stretch_objs/link_lift.obj
- link link_mast: geometry collision mesh filename=./stretch_objs/link_mast_collision.obj; visual mesh filename=./stretch_objs/link_mast.obj
- link link_right_wheel: geometry collision mesh filename=./stretch_objs/link_right_wheel_collision.obj; visual mesh filename=./stretch_objs/link_right_wheel.obj
- link link_wrist_pitch: geometry collision mesh filename=./stretch_objs/link_DW3_wrist_pitch_collision.obj; visual mesh filename=./stretch_objs/link_DW3_wrist_pitch.obj
- link link_wrist_roll: geometry collision mesh filename=./stretch_objs/link_DW3_wrist_roll_collision.obj; visual mesh filename=./stretch_objs/link_DW3_wrist_roll.obj
- link link_wrist_yaw: geometry collision mesh filename=./stretch_objs/link_wrist_yaw_collision.obj; visual mesh filename=./stretch_objs/link_wrist_yaw.obj
- link link_wrist_yaw_bottom: geometry collision mesh filename=./stretch_objs/link_DW3_wrist_yaw_bottom_collision.obj; visual mesh filename=./stretch_objs/link_DW3_wrist_yaw_bottom.obj
- link respeaker_base: geometry collision mesh filename=./stretch_objs/respeaker_base.obj; visual mesh filename=./stretch_objs/respeaker_base.obj
Joints:
- joint joint_gripper_finger_left: limit lower=0 upper=0 effort=0 velocity=0 -> lower=-0.0000000001 upper=0.0000000001 effort=0 velocity=0
- joint joint_gripper_finger_right: limit lower=0 upper=0 effort=0 velocity=0 -> lower=-0.0000000001 upper=0.0000000001 effort=0 velocity=0
